File: kicad/PressureSensor.kicad_pcb (KiCad board)
At the start: 2 copper layers, 2 parts

Commit message: update PCB layout
Parts:
- removed HX710: ~, Package_SO:SOIC-8_5.23x5.23mm_P1.27mm
- removed SENSOR1: ~, Library:pressure-sensor-SOIC-6
- added C2: .1u, Capacitor_SMD:C_0805_2012Metric_Pad1.18x1.45mm_HandSolder, F.Cu at (122.9, 91.2)
- added C3: .1u, Capacitor_SMD:C_0805_2012Metric_Pad1.18x1.45mm_HandSolder, F.Cu at (135.9, 84.8)
- added C4: .1u, Capacitor_SMD:C_0805_2012Metric_Pad1.18x1.45mm_HandSolder, F.Cu at (108.0, 84.5)
- added C5: .1u, Capacitor_SMD:C_0805_2012Metric_Pad1.18x1.45mm_HandSolder, F.Cu at (120.9, 68.3)
- added D1: STATUS, LED_SMD:LED_0805_2012Metric_Pad1.15x1.40mm_HandSolder, F.Cu at (131.1, 76.7)
- added FB1: FerriteBead_Small, Resistor_SMD:R_0805_2012Metric_Pad1.20x1.40mm_HandSolder, F.Cu at (107.3, 99.7)
- added FB2: FerriteBead_Small, Resistor_SMD:R_0805_2012Metric_Pad1.20x1.40mm_HandSolder, F.Cu at (128.0, 84.8)
- added J1: PROG, Connector_PinHeader_2.54mm:PinHeader_1x05_P2.54mm_Vertical, F.Cu at (104.8, 69.2)
- added POWER: USB_B_Micro, Connector_USB:USB_Micro-B_Amphenol_10118193-0001LF_Horizontal, F.Cu at (113.5, 106.0)
- added R1: 1k, Resistor_SMD:R_0805_2012Metric_Pad1.20x1.40mm_HandSolder, F.Cu at (122.9, 87.1)
- added R2: 1k, Resistor_SMD:R_0805_2012Metric_Pad1.20x1.40mm_HandSolder, F.Cu at (123.0, 95.0)
- added R3: 10k, Resistor_SMD:R_0805_2012Metric_Pad1.20x1.40mm_HandSolder, F.Cu at (135.4, 76.7)
- added R4: 1k, Resistor_SMD:R_0805_2012Metric_Pad1.20x1.40mm_HandSolder, F.Cu at (112.0, 83.8)
- added REF**: MountingHole_2.5mm, MountingHole:MountingHole_2.5mm, F.Cu at (136.5, 54.0)
- added REF**: MountingHole_2.5mm, MountingHole:MountingHole_2.5mm, F.Cu at (104.8, 54.0)
- added REF**: MountingHole_2.5mm, MountingHole:MountingHole_2.5mm, F.Cu at (104.8, 104.8)
- added REF**: MountingHole_2.5mm, MountingHole:MountingHole_2.5mm, F.Cu at (136.5, 104.8)
- added RESET: SW_Push, Button_Switch_THT:SW_PUSH_6mm_H5mm, F.Cu at (123.1, 99.3)
- added U1: SENSOR, Library:pressure-sensor-SOIC-6, F.Cu at (112.3, 89.9)
- added U2: HX710, Package_SO:SSOP-8_3.9x5.05mm_P1.27mm, F.Cu at (131.9, 89.0)
- added U3: DISPLAY, Library:7_seg_display_DIP12, F.Cu at (120.7, 58.4)
- added U4: AVR64DD32, Package_QFP:TQFP-32_7x7mm_P0.8mm, F.Cu at (119.8, 75.8)
Routing:
- net VCC: track 0.00 -> 95.2 mm, vias 0 -> 2
- net SPI_CLK: track 0.00 -> 46.8 mm, vias 0 -> 4
- net DIG_3: track 0.00 -> 46.1 mm, vias 0 -> 2
- net Net-(U4-PF5): track 0.00 -> 42.5 mm, vias 0 -> 2
- net SEG_B: track 0.00 -> 41.1 mm, vias 0 -> 3
- net SPI_MISO: track 0.00 -> 40.9 mm, vias 0 -> 4
- net DIG_4: track 0.00 -> 36.6 mm, vias 0 -> 2
- net SEG_A: track 0.00 -> 33.5 mm, vias 0 -> 1
- net DIG_1: track 0.00 -> 33.4 mm, vias 0 -> 1
- net SEG_E: track 0.00 -> 31.6 mm, vias 0 -> 1
- net DIG_2: track 0.00 -> 28.4 mm, vias 0 -> 2
- net SEG_C: track 0.00 -> 28.3 mm, vias 0 -> 3
- net SEG_D: track 0.00 -> 27.6 mm, vias 0 -> 1
- net UPDI: track 0.00 -> 26.6 mm, vias 0 -> 3
- net SEG_F: track 0.00 -> 26.1 mm, vias 0 -> 1
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- added copper zone on B.Cu, net GND
Other:
- board outline added: 38.1 x 57.2 mm
- board text added: "DAC"
- board text added: "GND"
- board text added: "JLCJLCJLCJLC"
- board text added: "Pressure Sensor @swharden v1.0"
- board text added: "SENSOR"
- board text added: "TX"
- board text added: "UPDI"
- board text added: "VCC"
