File: builds/2.0/kicad/PressureSensor.kicad_sch (KiCad schematic)
At the start: 25 parts, among them J1 USB_C_Receptacle_PowerOnly_6P, J2 PROG, U1 SENSOR, U2 HX710, U3 DISPLAY, U4 AVR64DD32

Commit message: update libraries
Parts:
- J1: footprint Connector_USB:USB_C_Receptacle_GCT_USB4105-xx-A_16P_TopMnt_Horizontal -> AAA_CUSTOM_LIBRARY:USB_C_Receptacle_GCT_USB4105-xx-A_16P_TopMnt_Horizontal
- U1: footprint Library:pressure-sensor-SOIC-6 -> AAA_CUSTOM_LIBRARY:pressure-sensor-SOIC-6
- U3: footprint Library:7_seg_display_DIP12 -> AAA_CUSTOM_LIBRARY:7_seg_display_DIP12
Changed lines of the file:
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@@
       (effects (font (size 1.27 1.27)))
     )
-    (property "Footprint" "Library:pressure-sensor-SOIC-6" (at 52.07 96.52 0)
+    (property "Footprint" "AAA_CUSTOM_LIBRARY:pressure-sensor-SOIC-6" (at 52.07 96.52 0)
       (effects (font (size 1.27 1.27)) hide)
     )
@@
       (effects (font (size 1.27 1.27)))
     )
-    (property "Footprint" "Library:7_seg_display_DIP12" (at 127.635 31.115 0)
+    (property "Footprint" "AAA_CUSTOM_LIBRARY:7_seg_display_DIP12" (at 127.635 31.115 0)
       (effects (font (size 1.27 1.27)) hide)
     )
@@
       (effects (font (size 1.27 1.27)))
     )
-    (property "Footprint" "Connector_USB:USB_C_Receptacle_GCT_USB4105-xx-A_16P_TopMnt_Horizontal" (at 41.275 40.64 0)
-      (effects (font (size 1.27 1.27)) hide)
-    )
+    (property "Footprint" "AAA_CUSTOM_LIBRARY:USB_C_Receptacle_GCT_USB4105-xx-A_16P_TopMnt_Horizontal" (at 41.275 40.64 0)
+      (effects (font (size 1.27 1.27)) hide)
+    )
