File: builds/2.0/kicad/PressureSensor.kicad_pcb (KiCad board)
At the start: 2 copper layers, 40.6 x 63.5 mm, 25 parts, among them J1 USB_C_Receptacle_PowerOnly_6P, J2 PROG, U1 SENSOR, U2 HX710, U3 DISPLAY, U4 AVR64DD32

Commit message: update pcb
Parts:
- moved R1 2.92 mm to (160.0, 102.6)
- moved R2 2.92 mm to (185.4, 102.9)
- moved C3 1.09 mm to (172.1, 76.1)
Routing:
- net VCC: track 115.1 -> 111.8 mm
- net BTN1: track 46.1 -> 48.9 mm
- net BTN2: track 40.6 -> 38.1 mm
- net Net-(J1-CC1): track 21.6 -> 19.1 mm
- net LED3: track 19.5 -> 18.5 mm
- net Net-(FB1-Pad1): track 10.9 -> 10.2 mm
- net Net-(J1-CC2): track 19.9 -> 19.4 mm
Other:
- board text removed: "SENSOR"
